File: hardware/cut down control board.kicad_pcb (KiCad board)
At the start: 2 copper layers, 152.4 x 63.7 mm, 52 parts, among them J1 CUTTER, J10 SAT(10 picoblade), J11 VGPS SELECT, J12 Analog In, J13 EXT BATT, J14 D8 I/O, J2 MOTOR, J3 ISP, J5 SAT(PIN HDR), J6 GPS(PIN HDR)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

Commit message: final board 10/12/2022
Parts:
- moved BT2 1.14 mm to (197.3, 81.6)
