File: hardware/cut down control board.kicad_sch (KiCad schematic)
At the start: 46 parts, among them J1 Conn_01x02, J2 Conn_01x02, J3 AVR-ISP-6, J4 Conn_01x02, J5 Conn_01x06_Female, J6 Conn_01x04_Female, J7 Conn_01x06_Male, J8 Conn_01x02, J9 Conn_01x06, M1 Motor_DC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

Commit message: More updates to PCB
Parts:
- added J10: SAT(10 picoblade), Connector_Molex:Molex_PicoBlade_53047-1010_1x10_P1.25mm_Vertical, symbol Connector:Conn_01x10_Female
- added J11: VGPS SELECT, Jumper:SolderJumper-3_P1.3mm_Bridged12_RoundedPad1.0x1.5mm, symbol Jumper:SolderJumper_3_Bridged12
- C10, C11, C3, C4, C5, C6, C7, C8, C9: footprint (none) -> Capacitor_THT:C_Axial_L5.1mm_D3.1mm_P7.50mm_Horizontal
- J1: value Conn_01x02 -> CUTTER; footprint Connector_PinHeader_2.54mm:PinHeader_1x02_P2.54mm_Vertical -> Connector_JST:JST_XH_B2B-XH-A_1x02_P2.50mm_Vertical
- J2: value Conn_01x02 -> MOTOR
- J4, J8: value Conn_01x02 -> Housing
- J5: value Conn_01x06_Female -> SAT(PIN HDR)
- J6: value Conn_01x04_Female -> GPS(PIN HDR); footprint (none) -> Connector_PinSocket_2.54mm:PinSocket_1x04_P2.54mm_Vertical
- J7: value Conn_01x06_Male -> DBG TTL
- J9: value Conn_01x06 -> GPS(JST SH)
- R1, R5: footprint (none) -> Resistor_THT:R_Axial_DIN0309_L9.0mm_D3.2mm_P12.70mm_Horizontal
- U6: footprint (none) -> Package_TO_SOT_THT:TO-220-3_Horizontal_TabDown
Connections:
- net +3.3V: now also J11.3 (B); no longer J6.3 (Pin_3)
- net +5V: now also J10.8 (Pin_8), J11.1 (A); no longer J9.2 (Pin_2)
- net GND: now also Q1.3 (S), R2.2, J10.10 (Pin_10)
- net RING: now also J10.5 (Pin_5)
- net RX_GPS: now also J6.3 (Pin_3); no longer J6.2 (Pin_2)
- net RX_SAT: now also J10.1 (Pin_1)
- net SLEEP: now also J10.7 (Pin_7)
- net TX_GPS: now also J6.2 (Pin_2); no longer J6.1 (Pin_1)
- net TX_SAT: now also J10.6 (Pin_6)
- net at C2.1, U1.10 (XTAL2/PB7): now also Y1.1
- net at C1.1, U1.9 (XTAL1/PB6): now also Y1.2
- new net +VGPS: J11.2 (C), J6.1 (Pin_1), J9.2 (Pin_2)
- new net CTS: J10.2 (Pin_2)
- new net Li_Ion: J10.9 (Pin_9)
- new net NetAv: J10.4 (Pin_4)
- new net RTS: J10.3 (Pin_3)
Other:
- note added: "GPS"
- note added: "I2C sensors"
- note added: "ISP and Debug"
- note added: "Indicators"
- note added: "MCU and MOSFETs"
- note added: "Power Supply"
- note added: "Rockblock"
- moved on the sheet: BT1, BT2, BT3, C1, C10, C11, C12, C2, C3, C4, C5, C6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

Commit message: board layout
Parts:
- D1: value LED, RED -> RED
- D2: value LED, GREEN -> GRN
- R1, R2, R3, R4, R5, R8, R9: footprint Resistor_THT:R_Axial_DIN0309_L9.0mm_D3.2mm_P12.70mm_Horizontal -> Resistor_THT:R_Axial_DIN0204_L3.6mm_D1.6mm_P7.62mm_Horizontal
- R6, R7: footprint Resistor_THT:R_Axial_DIN0207_L6.3mm_D2.5mm_P7.62mm_Horizontal -> Resistor_THT:R_Axial_DIN0204_L3.6mm_D1.6mm_P7.62mm_Horizontal
Connections:
- net +3.3V: now also R1.1

Commit message: finished board, generated gerbers
Parts:
- removed C3: 100nF, Capacitor_THT:C_Axial_L5.1mm_D3.1mm_P7.50mm_Horizontal, symbol Device:C_Small
- added J12: Analog In, Connector_PinHeader_2.54mm:PinHeader_2x03_P2.54mm_Vertical, symbol Connector_Generic:Conn_02x03_Odd_Even
- added SW1: SW_SPST, Connector_JST:JST_XH_B2B-XH-A_1x02_P2.50mm_Vertical, symbol Switch:SW_SPST
- J2: footprint Connector_JST:JST_XH_B2B-XH-AM_1x02_P2.50mm_Vertical -> Connector_JST:JST_XH_B2B-XH-A_1x02_P2.50mm_Vertical
- J3: value AVR-ISP-6 -> ISP
- J6: footprint Connector_PinSocket_2.54mm:PinSocket_1x04_P2.54mm_Vertical -> Connector_PinHeader_2.54mm:PinHeader_1x04_P2.54mm_Vertical
Connections:
- net +3.3V: now also J11.1 (A); no longer J11.3 (B)
- net +5V: now also J11.3 (B); no longer J11.1 (A)
- net +9V: now also SW1.2 (B); no longer BT1.1 (+), J1.1 (Pin_1), J2.1 (Pin_1)
- net GND: now also J12.2 (Pin_2), J12.4 (Pin_4), J12.6 (Pin_6)
- net RX_DBG: now also U1.16 (PB2); no longer U1.12 (PD6)
- net RX_GPS: now also U1.12 (PD6); no longer U1.16 (PB2)
- net TX_DBG: now also U1.15 (PB1); no longer U1.13 (PD7)
- net TX_GPS: now also U1.13 (PD7); no longer U1.15 (PB1)
- net A0: now reaches U1.23 (PC0)
- net A0: now also J12.1 (Pin_1)
- net A1: now reaches U1.24 (PC1)
- net A1: now also J12.3 (Pin_3)
- net A2: now reaches U1.25 (PC2)
- net A2: now also J12.5 (Pin_5)
- new net VDD: BT1.1 (+), J1.1 (Pin_1), J2.1 (Pin_1), SW1.1 (A)
- no-connect marks 7 -> 4
Other:
- moved on the sheet: BT1, BT2, BT3, C4, C6, C7, C8, C9, J11, J6, J9, R4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

Commit message: Added graphics, D8 input, and external power connector
Parts:
- added J13: EXT BATT, Connector_JST:JST_XH_B2B-XH-A_1x02_P2.50mm_Vertical, symbol Connector_Generic:Conn_01x02
- added J14: D8 I/O, Connector_JST:JST_XH_B2B-XH-A_1x02_P2.50mm_Vertical, symbol Connector_Generic:Conn_01x02
Connections:
- net GND: now also J13.2 (Pin_2), J14.2 (Pin_2)
- net VDD: now also J13.1 (Pin_1)
- net at U1.14 (PB0): now also J14.1 (Pin_1)
- no-connect marks 4 -> 3
Changed lines of the file:
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@@
   (title_block
     (title "${TITLE}")
-    (date "2022-09-22")
+    (date "2022-10-11")
     (rev "1")
     (company "Designed for the National Severe Storms Laboratory by Douglas Kennedy")
@@
   (junction (at 127 62.23) (diameter 0) (color 0 0 0 0)
   )
+  (junction (at 48.26 231.14) (diameter 0) (color 0 0 0 0)
+  )
   (junction (at 119.38 208.28) (diameter 0) (color 0 0 0 0)
   )
@@
   (no_connect (at 372.11 105.41))
   (no_connect (at 372.11 102.87))
-  (no_connect (at 78.74 45.72))
   (bus_entry (at 347.98 205.74) (size 2.54 -2.54)
     (stroke (width 0) (type default) (color 0 0 0 0))
@@
     (stroke (width 0) (type default) (color 0 0 0 0))
   )
+  (wire (pts (xy 48.26 231.14) (xy 49.53 231.14))
+    (stroke (width 0) (type default) (color 0 0 0 0))
+  )
   (wire (pts (xy 331.47 203.2) (xy 342.9 203.2))
     (stroke (width 0) (type default) (color 0 0 0 0))
@@
     (stroke (width 0) (type default) (color 0 0 0 0))
   )
+  (wire (pts (xy 48.26 233.68) (xy 48.26 240.03))
+    (stroke (width 0) (type default) (color 0 0 0 0))
+  )
   (polyline (pts (xy 165.1 152.4) (xy 165.1 190.5))
     (stroke (width 0) (type default) (color 0 0 0 0))
@@
     (stroke (width 0) (type default) (color 0 0 0 0))
   )
+  (wire (pts (xy 48.26 224.79) (xy 48.26 231.14))
+    (stroke (width 0) (type default) (color 0 0 0 0))
+  )
   (wire (pts (xy 142.24 245.11) (xy 142.24 246.38))
     (stroke (width 0) (type default) (color 0 0 0 0))
@@
     (stroke (width 0) (type default) (color 0 0 0 0))
   )
+  (wire (pts (xy 78.74 45.72) (xy 99.06 45.72))
+    (stroke (width 0) (type default) (color 0 0 0 0))
+  )
   (bus (pts (xy 252.73 237.49) (xy 252.73 240.03))
     (stroke (width 0) (type default) (color 0 0 0 0))
@@
   )
   (wire (pts (xy 78.74 81.28) (xy 86.36 81.28))
+    (stroke (width 0) (type default) (color 0 0 0 0))
+  )
+  (wire (pts (xy 99.06 48.26) (xy 99.06 49.53))
     (stroke (width 0) (type default) (color 0 0 0 0))
   )
@@
     )
     (property "Datasheet" "~" (id 3) (at 85.09 220.98 0)
+      (effects (font (size 1.27 1.27)) hide)
+    )
+    (pin "1")
+    (pin "2")
+  )
+  (symbol (lib_id "Connector_Generic:Conn_01x02") (at 104.14 45.72 0) (unit 1)
+    (in_bom yes) (on_board yes)
+    (property "Reference" "J14" (id 0) (at 102.87 40.64 0)
+      (effects (font (size 1.27 1.27)) (justify left))
+    )
+    (property "Value" "D8 I/O" (id 1) (at 102.87 43.18 0)
+      (effects (font (size 1.27 1.27)) (justify left))
+    )
+    (property "Footprint" "Connector_JST:JST_XH_B2B-XH-A_1x02_P2.50mm_Vertical" (id 2) (at 104.14 45.72 0)
+      (effects (font (size 1.27 1.27)) hide)
+    )
+    (property "Datasheet" "~" (id 3) (at 104.14 45.72 0)
       (effects (font (size 1.27 1.27)) hide)
     )
@@
     (pin "2")
   )
+  (symbol (lib_id "power:GND") (at 99.06 49.53 0) (unit 1)
+    (in_bom yes) (on_board yes) (fields_autoplaced)
+    (property "Reference" "#PWR0129" (id 0) (at 99.06 55.88 0)
+      (effects (font (size 1.27 1.27)) hide)
+    )
+    (property "Value" "GND" (id 1) (at 99.06 54.61 0))
+    (property "Footprint" "" (id 2) (at 99.06 49.53 0)
+      (effects (font (size 1.27 1.27)) hide)
+    )
+    (property "Datasheet" "" (id 3) (at 99.06 49.53 0)
+      (effects (font (size 1.27 1.27)) hide)
+    )
+    (pin "1")
+  )
   (symbol (lib_id "Device:C_Small") (at 252.73 69.85 0) (unit 1)
     (in_bom yes) (on_board yes) (fields_autoplaced)
@@
     (pin "1")
   )
+  (symbol (lib_id "Connector_Generic:Conn_01x02") (at 53.34 231.14 0) (unit 1)
+    (in_bom yes) (on_board yes)
+    (property "Reference" "J13" (id 0) (at 52.07 226.06 0)
+      (effects (font (size 1.27 1.27)) (justify left))
+    )
+    (property "Value" "EXT BATT" (id 1) (at 52.07 228.6 0)
+      (effects (font (size 1.27 1.27)) (justify left))
+    )
+    (property "Footprint" "Connector_JST:JST_XH_B2B-XH-A_1x02_P2.50mm_Vertical" (id 2) (at 53.34 231.14 0)
+      (effects (font (size 1.27 1.27)) hide)
+    )
+    (property "Datasheet" "~" (id 3) (at 53.34 231.14 0)
+      (effects (font (size 1.27 1.27)) hide)
+    )
+    (pin "1")
+    (pin "2")
+  )
   (symbol (lib_id "power:GND") (at 67.31 -54.61 0) (unit 1)
     (in_bom yes) (on_board yes) (fields_autoplaced)
@@
     )
     (property "Datasheet" "" (id 3) (at 116.84 237.49 0)
+      (effects (font (size 1.27 1.27)) hide)
+    )
+    (pin "1")
+  )
+  (symbol (lib_id "power:GND") (at 48.26 240.03 0) (unit 1)
+    (in_bom yes) (on_board yes) (fields_autoplaced)
+    (property "Reference" "#PWR0128" (id 0) (at 48.26 246.38 0)
+      (effects (font (size 1.27 1.27)) hide)
+    )
+    (property "Value" "GND" (id 1) (at 48.26 245.11 0))
+    (property "Footprint" "" (id 2) (at 48.26 240.03 0)
+      (effects (font (size 1.27 1.27)) hide)
+    )
+    (property "Datasheet" "" (id 3) (at 48.26 240.03 0)
       (effects (font (size 1.27 1.27)) hide)
     )
@@
     (pin "3")
   )
+  (symbol (lib_id "power:VDD") (at 48.26 224.79 0) (unit 1)
+    (in_bom yes) (on_board yes) (fields_autoplaced)
+    (property "Reference" "#PWR0125" (id 0) (at 48.26 228.6 0)
+      (effects (font (size 1.27 1.27)) hide)
+    )
+    (property "Value" "VDD" (id 1) (at 48.26 219.71 0))
+    (property "Footprint" "" (id 2) (at 48.26 224.79 0)
+      (effects (font (size 1.27 1.27)) hide)
+    )
+    (property "Datasheet" "" (id 3) (at 48.26 224.79 0)
+      (effects (font (size 1.27 1.27)) hide)
+    )
+    (pin "1")
+  )
   (symbol (lib_id "power:+3.3V") (at 274.32 200.66 0) (unit 1)
     (in_bom yes) (on_board yes) (fields_autoplaced)
@@
       (reference "#PWR0124") (unit 1) (value "+3.3V") (footprint "")
     )
+    (path "/d428702e-0fdc-4806-bc7e-baaa2fb202ec"
+      (reference "#PWR0125") (unit 1) (value "VDD") (footprint "")
+    )
     (path "/a24eb835-9610-4b64-b2f8-4810650eebf3"
       (reference "#PWR0126") (unit 1) (value "GND") (footprint "")
@@
       (reference "#PWR0127") (unit 1) (value "GND") (footprint "")
     )
+    (path "/6c577a44-6a55-45c1-9de2-98ee737bb956"
+      (reference "#PWR0128") (unit 1) (value "GND") (footprint "")
+    )
+    (path "/46f1da9d-e4f7-4f59-8d68-e6b75f598bb9"
+      (reference "#PWR0129") (unit 1) (value "GND") (footprint "")
+    )
     (path "/56fd23ba-f276-457e-9d47-ead56b5f10ae"
       (reference "BT1") (unit 1) (value "Battery_Cell") (footprint "doug_Library:BatteryHolder_Keystone_1051_1xCR123A")
@@
       (reference "J12") (unit 1) (value "Analog In") (footprint "Connector_PinHeader_2.54mm:PinHeader_2x03_P2.54mm_Vertical")
     )
+    (path "/64c409ce-b55c-4fd1-9510-5a84debb280c"
+      (reference "J13") (unit 1) (value "EXT BATT") (footprint "Connector_JST:JST_XH_B2B-XH-A_1x02_P2.50mm_Vertical")
+    )
+    (path "/39b0e5b6-fc85-4735-aa86-6938082c378e"
+      (reference "J14") (unit 1) (value "D8 I/O") (footprint "Connector_JST:JST_XH_B2B-XH-A_1x02_P2.50mm_Vertical")
+    )
     (path "/78b7f654-0f2f-4de3-bb02-2c8ac291eb64"

Commit message: final board 10/12/2022
Other:
- moved on the sheet: C10, C11, C12, C5, J11, J3, J6, J7, J9, R8, R9, U2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

Commit message: flipped motor down
Parts:
- R6, R7: value 330 -> 130
Changed lines of the file:
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@@
     (in_bom yes) (on_board yes) (fields_autoplaced)
     (property "Reference" "R7" (id 0) (at 78.74 171.45 90))
-    (property "Value" "330" (id 1) (at 78.74 173.99 90))
+    (property "Value" "130" (id 1) (at 78.74 173.99 90))
     (property "Footprint" "Resistor_THT:R_Axial_DIN0204_L3.6mm_D1.6mm_P7.62mm_Horizontal" (id 2) (at 78.994 176.784 90)
       (effects (font (size 1.27 1.27)) hide)
@@
     (in_bom yes) (on_board yes) (fields_autoplaced)
     (property "Reference" "R6" (id 0) (at 78.74 160.02 90))
-    (property "Value" "330" (id 1) (at 78.74 162.56 90))
+    (property "Value" "130" (id 1) (at 78.74 162.56 90))
     (property "Footprint" "Resistor_THT:R_Axial_DIN0204_L3.6mm_D1.6mm_P7.62mm_Horizontal" (id 2) (at 78.994 165.354 90)
       (effects (font (size 1.27 1.27)) hide)
@@
     )
     (path "/d05a1d79-dcc9-4028-a0b5-0f7a5193ca97"
-      (reference "R6") (unit 1) (value "330") (footprint "Resistor_THT:R_Axial_DIN0204_L3.6mm_D1.6mm_P7.62mm_Horizontal")
+      (reference "R6") (unit 1) (value "130") (footprint "Resistor_THT:R_Axial_DIN0204_L3.6mm_D1.6mm_P7.62mm_Horizontal")
     )
     (path "/76db2041-e8da-40ae-9341-8e0a72bcb539"
-      (reference "R7") (unit 1) (value "330") (footprint "Resistor_THT:R_Axial_DIN0204_L3.6mm_D1.6mm_P7.62mm_Horizontal")
+      (reference "R7") (unit 1) (value "130") (footprint "Resistor_THT:R_Axial_DIN0204_L3.6mm_D1.6mm_P7.62mm_Horizontal")
     )
     (path "/20e0e586-8e15-4284-8969-64c6cd6a4458"

Commit message: reversed picoblade connector for rockblock 9603
cable pin 1 to pin 10, pin 2 to 9, etc (premade cables are reversed)
Connections:
- net +5V: now also J10.3 (Pin_3); no longer J10.8 (Pin_8)
- net CTS: now also J10.9 (Pin_9); no longer J10.2 (Pin_2)
- net GND: now also J10.1 (Pin_1); no longer J10.10 (Pin_10)
- net Li_Ion: now also J10.2 (Pin_2); no longer J10.9 (Pin_9)
- net NetAv: now also J10.7 (Pin_7); no longer J10.4 (Pin_4)
- net RING: now also J10.6 (Pin_6); no longer J10.5 (Pin_5)
- net RTS: now also J10.8 (Pin_8); no longer J10.3 (Pin_3)
- net RX_SAT: now also J10.10 (Pin_10); no longer J10.1 (Pin_1)
- net SLEEP: now also J10.4 (Pin_4); no longer J10.7 (Pin_7)
- net TX_SAT: now also J10.5 (Pin_5); no longer J10.6 (Pin_6)
Changed lines of the file:
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@@
     (effects (font (size 1.27 1.27)) (justify left bottom))
   )
-  (label "NetAv" (at 331.47 210.82 0)
+  (label "SLEEP" (at 331.47 210.82 0)
     (effects (font (size 1.27 1.27)) (justify left bottom))
   )
@@
     (effects (font (size 1.27 1.27)) (justify left bottom))
   )
-  (label "Li_Ion" (at 331.47 223.52 0)
+  (label "CTS" (at 331.47 223.52 0)
     (effects (font (size 1.27 1.27)) (justify left bottom))
   )
-  (label "+5V" (at 331.47 220.98 0)
+  (label "RTS" (at 331.47 220.98 0)
     (effects (font (size 1.27 1.27)) (justify left bottom))
   )
@@
     (effects (font (size 1.27 1.27)) (justify left bottom))
   )
-  (label "RX_SAT" (at 331.47 203.2 0)
+  (label "GND" (at 331.47 203.2 0)
     (effects (font (size 1.27 1.27)) (justify left bottom))
   )
@@
     (effects (font (size 1.27 1.27)) (justify left bottom))
   )
-  (label "RTS" (at 331.47 208.28 0)
+  (label "+5V" (at 331.47 208.28 0)
     (effects (font (size 1.27 1.27)) (justify left bottom))
   )
@@
     (effects (font (size 1.27 1.27)) (justify left bottom))
   )
-  (label "CTS" (at 331.47 205.74 0)
+  (label "Li_Ion" (at 331.47 205.74 0)
     (effects (font (size 1.27 1.27)) (justify left bottom))
   )
@@
     (effects (font (size 1.27 1.27)) (justify left bottom))
   )
-  (label "SLEEP" (at 331.47 218.44 0)
+  (label "NetAv" (at 331.47 218.44 0)
     (effects (font (size 1.27 1.27)) (justify left bottom))
   )
@@
     (effects (font (size 1.27 1.27)) (justify left bottom))
   )
-  (label "TX_SAT" (at 331.47 215.9 0)
+  (label "RING" (at 331.47 215.9 0)
     (effects (font (size 1.27 1.27)) (justify left bottom))
   )
@@
     (effects (font (size 1.27 1.27)) (justify left bottom))
   )
-  (label "RING" (at 331.47 213.36 0)
+  (label "TX_SAT" (at 331.47 213.36 0)
     (effects (font (size 1.27 1.27)) (justify left bottom))
   )
@@
     (effects (font (size 1.27 1.27)) (justify left bottom))
   )
-  (label "GND" (at 331.47 226.06 0)
+  (label "RX_SAT" (at 331.47 226.06 0)
     (effects (font (size 1.27 1.27)) (justify left bottom))
   )

Commit message: modify receiver plates
Connections:
- removed net SLEEP: J10.4 (Pin_4), J5.2 (Pin_2), U1.5 (PD3), U4. (VCC)
- no-connect marks 3 -> 7
Changed lines of the file:
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@@
   (junction (at 127 104.14) (diameter 0) (color 0 0 0 0)
   )
+  (no_connect (at 342.9 179.07))
+  (no_connect (at 342.9 210.82))
   (no_connect (at 370.84 118.11))
   (no_connect (at 370.84 110.49))
   (no_connect (at 370.84 107.95))
+  (no_connect (at 363.22 200.66))
+  (no_connect (at 78.74 96.52))
   (bus_entry (at 347.98 205.74) (size 2.54 -2.54)
     (stroke (width 0) (type default) (color 0 0 0 0))
@@
     (stroke (width 0) (type solid) (color 0 0 0 0))
   )
-  (bus_entry (at 350.52 203.2) (size 2.54 -2.54)
-    (stroke (width 0) (type solid) (color 0 0 0 0))
-  )
   (bus_entry (at 347.98 189.23) (size 2.54 2.54)
     (stroke (width 0) (type default) (color 0 0 0 0))
@@
     (stroke (width 0) (type default) (color 0 0 0 0))
   )
-  (wire (pts (xy 78.74 96.52) (xy 86.36 96.52))
-    (stroke (width 0) (type default) (color 0 0 0 0))
-  )
   (wire (pts (xy 38.1 38.1) (xy 38.1 35.56))
     (stroke (width 0) (type default) (color 0 0 0 0))
@@
     (stroke (width 0) (type default) (color 0 0 0 0))
   )
-  (wire (pts (xy 342.9 210.82) (xy 331.47 210.82))
-    (stroke (width 0) (type default) (color 0 0 0 0))
-  )
   (wire (pts (xy 226.06 238.76) (xy 234.95 238.76))
     (stroke (width 0) (type default) (color 0 0 0 0))
@@
     (stroke (width 0) (type default) (color 0 0 0 0))
   )
-  (wire (pts (xy 353.06 200.66) (xy 363.22 200.66))
-    (stroke (width 0) (type default) (color 0 0 0 0))
-  )
   (wire (pts (xy 78.74 106.68) (xy 86.36 106.68))
     (stroke (width 0) (type default) (color 0 0 0 0))
@@
   )
   (wire (pts (xy 133.35 246.38) (xy 142.24 246.38))
-    (stroke (width 0) (type default) (color 0 0 0 0))
-  )
-  (wire (pts (xy 336.55 179.07) (xy 342.9 179.07))
     (stroke (width 0) (type default) (color 0 0 0 0))
   )
@@
     (effects (font (size 3 3) bold) (justify left bottom))
   )
-  (label "SLEEP" (at 86.36 96.52 0)
-    (effects (font (size 1.27 1.27)) (justify left bottom))
-  )
   (label "TX_GPS" (at 86.36 106.68 0)
-    (effects (font (size 1.27 1.27)) (justify left bottom))
-  )
-  (label "SLEEP" (at 336.55 179.07 0)
-    (effects (font (size 1.27 1.27)) (justify left bottom))
-  )
-  (label "SLEEP" (at 331.47 210.82 0)
     (effects (font (size 1.27 1.27)) (justify left bottom))
   )
@@
     (effects (font (size 1.27 1.27)) (justify left bottom))
   )
-  (label "SLEEP" (at 355.6 200.66 0)
-    (effects (font (size 1.27 1.27)) (justify left bottom))
-  )
