File: hardware/cut down control board.kicad_sch (KiCad schematic)
At the start: 51 parts, among them J1 CUTTER, J10 SAT(10 picoblade), J11 VGPS SELECT, J12 Analog In, J13 EXT BATT, J14 D8 I/O, J2 MOTOR, J3 ISP, J4 Housing, J5 SAT(PIN HDR)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

Commit message: add PDF of pcb and schematic as produced
Parts:
- R4: value 100K -> 500K
- R5: value 33K -> 165K
Changed lines of the file:
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@@
       (effects (font (size 1.27 1.27)) (justify left))
     )
-    (property "Value" "100K" (id 1) (at 87.63 222.2499 0)
+    (property "Value" "500K" (id 1) (at 87.63 222.2499 0)
       (effects (font (size 1.27 1.27)) (justify left))
     )
@@
       (effects (font (size 1.27 1.27)) (justify left))
     )
-    (property "Value" "33K" (id 1) (at 87.63 232.4099 0)
+    (property "Value" "165K" (id 1) (at 87.63 232.4099 0)
       (effects (font (size 1.27 1.27)) (justify left))
     )
@@
     )
     (path "/31bb6f47-4193-47ce-9020-a52cb4daf773"
-      (reference "R4") (unit 1) (value "100K") (footprint "Resistor_THT:R_Axial_DIN0204_L3.6mm_D1.6mm_P7.62mm_Horizontal")
+      (reference "R4") (unit 1) (value "500K") (footprint "Resistor_THT:R_Axial_DIN0204_L3.6mm_D1.6mm_P7.62mm_Horizontal")
     )
     (path "/4bad86b4-5104-4646-ae38-1e166ce89fbe"
-      (reference "R5") (unit 1) (value "33K") (footprint "Resistor_THT:R_Axial_DIN0204_L3.6mm_D1.6mm_P7.62mm_Horizontal")
+      (reference "R5") (unit 1) (value "165K") (footprint "Resistor_THT:R_Axial_DIN0204_L3.6mm_D1.6mm_P7.62mm_Horizontal")
     )
     (path "/d05a1d79-dcc9-4028-a0b5-0f7a5193ca97"

Commit message: add wire lengths in schematic
Parts:
- M1: value Motor_DC -> Greartisan 250 RPM
- R10: value Nichrome -> Nichrome, 32 AWG, 3 ohm
- SW1: value SW_SPST -> MBZ101A01C02X02
Other:
- note added: "140mm"
- note added: "180mm"
- note added: "RED DOT"
- moved on the sheet: R4, R5, SW1
